Commit message: Added new realsense foxy description package, and updated the relevant documentation
Signed-off-by: Tan Jing Peng Glenn <glenn_tan@artc.a-star.edu.sg>

File: assets/environment/realsense2_description/urdf/_d415.urdf.xacro (robot description, xacro)
@@ -3,5 +3,5 @@
 License: Apache 2.0. See LICENSE file in root directory.
 Copyright(c) 2017 Intel Corporation. All Rights Reserved
-This is the URDF model for the Intel RealSense 415 camera, in it's
+This is the URDF model for the Intel RealSense 415 camera, in its
 aluminum peripherial evaluation case.
 -->
@@ -9,5 +9,6 @@
   <!-- Includes -->
   <xacro:include filename="$(find realsense2_description)/urdf/_materials.urdf.xacro" />
-  <xacro:macro name="sensor_d415" params="parent *origin  name:=camera  use_nominal_extrinsics:=false">
+  <xacro:include filename="$(find realsense2_description)/urdf/_usb_plug.urdf.xacro" />
+  <xacro:macro name="sensor_d415" params="parent *origin  name:=camera  use_nominal_extrinsics:=false  add_plug:=false">
     <xacro:property name="M_PI" value="3.1415926535897931" />
     <!-- The following values are approximate, and the camera node
@@ -117,4 +118,9 @@
       <link name="${name}_color_optical_frame"/>
     </xacro:if>
+    <xacro:if value="$(arg add_plug)">
+      <xacro:usb_plug parent="${name}_link" name="${name}_usb_plug">
+        <origin xyz="${d415_cam_mount_from_center_offset - 0.01587} ${-d415_cam_depth_py - 0.0358} 0" rpy="0 0 0"/>
+      </xacro:usb_plug>
+    </xacro:if>
   </xacro:macro>
 </robot>

File: assets/environment/realsense2_description/urdf/_d435.urdf.xacro (robot description, xacro)
@@ -3,5 +3,5 @@
 License: Apache 2.0. See LICENSE file in root directory.
 Copyright(c) 2017 Intel Corporation. All Rights Reserved
-This is the URDF model for the Intel RealSense 430 camera, in it's
+This is the URDF model for the Intel RealSense 430 camera, in its
 aluminum peripherial evaluation case.
 -->
@@ -9,5 +9,7 @@
   <!-- Includes -->
   <xacro:include filename="$(find realsense2_description)/urdf/_materials.urdf.xacro" />
+  <xacro:include filename="$(find realsense2_description)/urdf/_usb_plug.urdf.xacro" />
   <xacro:macro name="sensor_d435" params="parent *origin name:=camera use_nominal_extrinsics:=false">
+    <xacro:arg name="add_plug" default="false" />
     <xacro:property name="M_PI" value="3.1415926535897931" />
     <!-- The following values are approximate, and the camera node
@@ -63,5 +65,5 @@
       <inertial>
         <!-- The following are not reliable values, and should not be used for modeling -->
-        <mass value="0.564" />
+        <mass value="0.072" />
         <origin xyz="0 0 0" />
         <inertia ixx="0.003881243" ixy="0.0" ixz="0.0" iyy="0.000498940" iyz="0.0" izz="0.003879257" />
@@ -123,4 +125,9 @@
       <link name="${name}_color_optical_frame"/>
     </xacro:if>
+    <xacro:if value="$(arg add_plug)">
+      <xacro:usb_plug parent="${name}_link" name="${name}_usb_plug">
+        <origin xyz="${d435_cam_mount_from_center_offset - 0.02095} ${-d435_cam_depth_py - 0.0353} 0" rpy="0 0 0"/>
+      </xacro:usb_plug>
+    </xacro:if>
   </xacro:macro>
 </robot>

File: scenes/ur5_test/urdf/scene.urdf.xacro (robot description, xacro)
@@ -19,5 +19,6 @@
  <xacro:include filename="$(find realsense2_description)/urdf/_d415.urdf.xacro"/>
  <xacro:arg name="use_nominal_extrinsics" default="true" />
- <xacro:sensor_d415 parent="table_" use_nominal_extrinsics="$(arg use_nominal_extrinsics)">
+ <xacro:arg name="add_plug" default="false" />
+ <xacro:sensor_d415 parent="table_" use_nominal_extrinsics="$(arg use_nominal_extrinsics)" add_plug="$(arg add_plug)">
 	<!--origin xyz="-0.6385 0.2 0.56" rpy="0 1.57079506 0"/-->
 	<origin xyz="-0.5 0.2 0.46" rpy="0 1.57079506 0"/>
